File: Debugger.kicad_sch (KiCad schematic)
At the start: 20 parts, among them J101 USB_B_Mini, J102 Conn_01x06_Pin, SW101 SW_SPDT, U101 STM32F103C8Tx

Commit message: ethernet, debugger and usb layouts re-designed
Parts:
- SW101: footprint footprints:SW_PTS636_SM43J_SMTR_LFS -> Button_Switch_SMD:SW_SPST_B3U-1000P
Changed lines of the file:
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@@
 			)
 		)
-		(property "Footprint" "footprints:SW_PTS636_SM43J_SMTR_LFS"
+		(property "Footprint" "Button_Switch_SMD:SW_SPST_B3U-1000P"
 			(at 98.0438 48.8381 0)
 			(effects

Commit message: some additions
Parts:
- renumbered C108 to C?, C102 to C?, C111 to C?, C105 to C?, C103 to C?, C106 to C?, C107 to C?, C104 to C?, C101 to C?, C110 to C?, C109 to C?, J102 to J?, J101 to J?, R105 to R?, R102 to R?, R101 to R?, R104 to R?, SW101 to SW?, U101 to U?, XTAL101 to XTAL?
