File: Motor_Driver1.kicad_sch (KiCad schematic)
At the start: 20 parts, among them J801 Conn_01x02_Socket, U801 DMHT6016LFJ-13, U802 DRV8701

Commit message: critical nets coloured,some tracks rerouted, section 9 completed.
Connections:
- net GND: now also U802.25 (GND)
Changed lines of the file:
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@@
 		(pin "5"
+		)
+		(pin "25"
 		)
 		(instances

Commit message: schematic pages are reviewed
Other:
- note added: "H-BRIDGE"
- note added: "MOTOR DRIVER 1"
- moved on the sheet: J801
