File: USB_to_TTL.kicad_sch (KiCad schematic)
At the start: 3 parts, among them J501 USB_B_Mini, U501 CH340C

Commit message: some additions
Parts:
- renumbered C501 to C?, J501 to J?, U501 to U?
Changed lines of the file:
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@@
 		(dnp no)
 		(fields_autoplaced yes)
-		(property "Reference" "U501"
+		(property "Reference" "U?"
 			(at 152.8191 111.76 0)
 			(effects
@@
 		)
 		(instances
-			(project ""
-				(path "/8a424437-6f3e-424c-a786-3b8b285eee60/eec587cf-a1a3-41c9-8f50-400433a25eba"
-					(reference "U501")
+			(project "mixed signal board project"
+				(path "/8a424437-6f3e-424c-a786-3b8b285eee60/00859c04-2135-4e2f-827b-32ca1cdd4b39/95928e7c-f6d0-4a41-860c-c50b4c0b320e"
+					(reference "U?")
 					(unit 1)
 				)
@@
 		(dnp no)
 		(fields_autoplaced yes)
-		(property "Reference" "#PWR0503"
+		(property "Reference" "#PWR0612"
 			(at 198.4227 120.2275 0)
 			(effects
@@
 		(instances
 			(project "mixed signal board project"
-				(path "/8a424437-6f3e-424c-a786-3b8b285eee60/eec587cf-a1a3-41c9-8f50-400433a25eba"
-					(reference "#PWR0503")
+				(path "/8a424437-6f3e-424c-a786-3b8b285eee60/00859c04-2135-4e2f-827b-32ca1cdd4b39/95928e7c-f6d0-4a41-860c-c50b4c0b320e"
+					(reference "#PWR0612")
 					(unit 1)
 				)
@@
 		(dnp no)
 		(fields_autoplaced yes)
-		(property "Reference" "#PWR0501"
+		(property "Reference" "#PWR0610"
 			(at 133.7057 64.1264 0)
 			(effects
@@
 		)
 		(instances
-			(project ""
-				(path "/8a424437-6f3e-424c-a786-3b8b285eee60/eec587cf-a1a3-41c9-8f50-400433a25eba"
-					(reference "#PWR0501")
+			(project "mixed signal board project"
+				(path "/8a424437-6f3e-424c-a786-3b8b285eee60/00859c04-2135-4e2f-827b-32ca1cdd4b39/95928e7c-f6d0-4a41-860c-c50b4c0b320e"
+					(reference "#PWR0610")
 					(unit 1)
 				)
@@
 		(dnp no)
 		(fields_autoplaced yes)
-		(property "Reference" "J501"
+		(property "Reference" "J?"
 			(at 204.47 96.9993 0)
 			(effects
@@
 		)
 		(instances
-			(project ""
-				(path "/8a424437-6f3e-424c-a786-3b8b285eee60/eec587cf-a1a3-41c9-8f50-400433a25eba"
-					(reference "J501")
+			(project "mixed signal board project"
+				(path "/8a424437-6f3e-424c-a786-3b8b285eee60/00859c04-2135-4e2f-827b-32ca1cdd4b39/95928e7c-f6d0-4a41-860c-c50b4c0b320e"
+					(reference "J?")
 					(unit 1)
 				)
@@
 		(on_board yes)
 		(dnp no)
-		(property "Reference" "C501"
+		(property "Reference" "C?"
 			(at 136.3872 69.3488 0)
 			(effects
@@
 		)
 		(instances
-			(project ""
-				(path "/8a424437-6f3e-424c-a786-3b8b285eee60/eec587cf-a1a3-41c9-8f50-400433a25eba"
-					(reference "C501")
+			(project "mixed signal board project"
+				(path "/8a424437-6f3e-424c-a786-3b8b285eee60/00859c04-2135-4e2f-827b-32ca1cdd4b39/95928e7c-f6d0-4a41-860c-c50b4c0b320e"
+					(reference "C?")
 					(unit 1)
 				)
@@
 		(dnp no)
 		(fields_autoplaced yes)
-		(property "Reference" "#PWR0502"
+		(property "Reference" "#PWR0611"
 			(at 140.5506 83.8845 0)
 			(effects
@@
 		)
 		(instances
-			(project ""
-				(path "/8a424437-6f3e-424c-a786-3b8b285eee60/eec587cf-a1a3-41c9-8f50-400433a25eba"
-					(reference "#PWR0502")
-					(unit 1)
-				)
+			(project "mixed signal board project"
+				(path "/8a424437-6f3e-424c-a786-3b8b285eee60/00859c04-2135-4e2f-827b-32ca1cdd4b39/95928e7c-f6d0-4a41-860c-c50b4c0b320e"
+					(reference "#PWR0611")
+					(unit 1)
+				)
