File: ethernet.kicad_sch (KiCad schematic)
At the start: 32 parts, among them J201 8P8C_Shielded, SW201 SW_SPDT, U201 DP83826ERHBR, Y201 25Mhz

Commit message: schematic pages are reviewed
Parts:
- renumbered R208 to R207, R207 to R208
Other:
- note added: "*If needed"
- note added: "EXTERNAL PULL-UP TO MDIO PIN"
