File: mixed signal board project.kicad_sch (KiCad schematic)
At the start: 0 parts

Commit message: I2C pins that is on ADC and DAC corrected
Other:
- sheet ADC ports: added SCL, SDA; removed SCK_ADC, SDA_ADC
- sheet DAC adn MIC ports: added SCL, SDA; removed SCL_DAC, SDA_DAC
- sheet STM32F407 ports: added SCL, SDA; removed SCK_ADC, SCL_DAC, SDA_ADC, SDA_DAC
Changed lines of the file:
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@@
 			)
 		)
-		(pin "SCL_DAC" input
+		(pin "SCL" input
 			(at 91.8099 109.4445 0)
 			(effects
@@
 			)
 		)
-		(pin "SDA_DAC" bidirectional
+		(pin "SDA" bidirectional
 			(at 91.8099 111.8149 0)
 			(effects
@@
 			)
 		)
-		(pin "SCL_DAC" output
+		(pin "SCL" output
 			(at 104.3039 109.1789 180)
 			(effects
@@
 			)
 		)
-		(pin "SDA_DAC" bidirectional
+		(pin "SDA" bidirectional
 			(at 104.3039 111.3912 180)
 			(effects
@@
 			)
 		)
-		(pin "SCK_ADC" output
+		(pin "SCL" output
 			(at 104.3039 139.877 180)
 			(effects
@@
 			)
 		)
-		(pin "SDA_ADC" bidirectional
+		(pin "SDA" bidirectional
 			(at 104.3039 142.2664 180)
 			(effects
@@
 			)
 		)
-		(pin "SCK_ADC" input
+		(pin "SCL" input
 			(at 84.756 145.408 0)
 			(effects
@@
 			)
 		)
-		(pin "SDA_ADC" bidirectional
+		(pin "SDA" bidirectional
 			(at 84.756 148.1735 0)
 			(effects

Commit message: some additions
Other:
- removed sheet ADC
- removed sheet DAC adn MIC
- removed sheet Debugger
- removed sheet Ethernet
- removed sheet Motor_Driver1
- removed sheet Motor_Driver2
- removed sheet Power Input and Regulators
- removed sheet STM32F407
- removed sheet USB_to_TTL
- added sheet Block_diagram (Block_diagram.kicad_sch)
- added sheet Block_schematics (Block_schematics.kicad_sch)
- added sheet Power_Budget (Power_Budget.kicad_sch)
- note added: "-ETHERNET -MOTOR DRIVERx2 -ADC & DAC & MIC -HEADPHONE & SPEAKER"
- note added: "MIXED SIGNAL BOARD PROJECT"
