File: ADC.kicad_sch (KiCad schematic)
At the start: 14 parts, among them J301 Conn_01x04_Pin, U301 ADS122C04IPW

Commit message: some design failures reviewed(MIC VDD is 1V8, Motor Drivers' pull-up to DVDD pin, I2C net fixed). Routing mostly done.
Connections:
- net SCK_ADC renamed SCL
- net SDA_ADC renamed SDA
Changed lines of the file:
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@@
 		)
 	)
-	(hierarchical_label "SCK_ADC"
+	(hierarchical_label "SCL"
 		(shape input)
 		(at 227.3156 82.4097 0)
@@
 		)
 	)
-	(hierarchical_label "SDA_ADC"
+	(hierarchical_label "SDA"
 		(shape bidirectional)
 		(at 226.9769 79.8693 0)

Commit message: some additions
Parts:
- renumbered C306 to C?, C305 to C?, C302 to C?, C303 to C?, C304 to C?, C301 to C?, FB301 to FB?, J301 to J?, R301 to R?, R305 to R?, R303 to R?, R302 to R?, R304 to R?, U301 to U?
